File: darksky-porch-light.kicad_pcb (KiCad board)
At the start: 2 copper layers, 15 parts, among them J1 Motion, J2 FTDI, Q1 QM6006D, U1 ESP32-WROOM-32E, U2 AD8606ARZ

Commit message: layout
Parts:
- added BT1: Battery_Cell, Battery:BatteryHolder_Keystone_3002_1x2032, F.Cu at (137.9, 117.1)
- added C1: 0.1uF, Capacitor_SMD:C_0603_1608Metric, F.Cu at (159.6, 108.6)
- added C11: 0.1uF, Capacitor_SMD:C_0603_1608Metric, F.Cu at (185.2, 101.0)
- added C12: 0.1uF, Capacitor_SMD:C_0603_1608Metric, F.Cu at (120.2, 81.2)
- added C13: 0.1uF, Capacitor_SMD:C_0603_1608Metric, F.Cu at (183.8, 96.8)
- added C14: 0.1uF, Capacitor_SMD:C_0603_1608Metric, F.Cu at (163.4, 106.0)
- added C2: 10uF, Capacitor_SMD:C_0603_1608Metric, F.Cu at (166.4, 107.6)
- added C3: 0.1uF, Capacitor_SMD:C_0603_1608Metric, F.Cu at (179.8, 108.6)
- added C4: 0.1uF, Capacitor_SMD:C_0603_1608Metric, F.Cu at (162.6, 130.8)
- added C5: 0.1uF, Capacitor_SMD:C_0603_1608Metric, F.Cu at (176.0, 116.8)
- added C6: 100uF, Capacitor_SMD:CP_Elec_6.3x5.4_Nichicon, F.Cu at (185.6, 79.2)
- added C7: 10uF, Capacitor_SMD:C_0603_1608Metric, F.Cu at (150.0, 104.0)
- added C8: 0.1uF, Capacitor_SMD:C_0603_1608Metric, F.Cu at (144.4, 95.0)
- added C9: 0.1uF, Capacitor_SMD:C_0603_1608Metric, F.Cu at (147.4, 98.8)
- added D10: 2200K, LED_SMD:LED_PLCC_2835_Handsoldering, B.Cu at (145.0, 95.0)
- added D11: 2200K, LED_SMD:LED_PLCC_2835_Handsoldering, B.Cu at (146.0, 90.0)
- added D12: 2200K, LED_SMD:LED_PLCC_2835_Handsoldering, B.Cu at (150.0, 86.0)
- added D13: LED, LED_SMD:LED_0603_1608Metric_Pad1.05x0.95mm_HandSolder, F.Cu at (171.4, 116.6)
- added D3: 2200K, LED_SMD:LED_PLCC_2835_Handsoldering, B.Cu at (164.0, 90.0)
- added D4: 2200K, LED_SMD:LED_PLCC_2835_Handsoldering, B.Cu at (165.0, 95.0)
- added D5: 2200K, LED_SMD:LED_PLCC_2835_Handsoldering, B.Cu at (164.0, 100.0)
- added D6: 2200K, LED_SMD:LED_PLCC_2835_Handsoldering, B.Cu at (160.0, 104.0)
- added D7: 2200K, LED_SMD:LED_PLCC_2835_Handsoldering, B.Cu at (155.0, 105.0)
- added D8: 2200K, LED_SMD:LED_PLCC_2835_Handsoldering, B.Cu at (150.0, 104.0)
- added D9: 2200K, LED_SMD:LED_PLCC_2835_Handsoldering, B.Cu at (146.0, 100.0)
- added F1: Fuse, Fuse:Fuseholder_Littelfuse_Nano2_154x, F.Cu at (144.8, 61.4)
- added H1: M3, MountingHole:MountingHole_3.2mm_M3, F.Cu at (155.0, 60.0)
- added H2: M3, MountingHole:MountingHole_3.2mm_M3, F.Cu at (120.0, 95.0)
- added H3: M3, MountingHole:MountingHole_3.2mm_M3, F.Cu at (155.0, 130.0)
- added H4: M3, MountingHole:MountingHole_3.2mm_M3, F.Cu at (190.0, 95.0)
- added J3: SM06B-GHS-TB, Connector_JST:JST_GH_SM06B-GHS-TB_1x06-1MP_P1.25mm_Horizontal, F.Cu at (170.6, 127.8)
- added J4: Motion, Connector_PinSocket_2.54mm:PinSocket_1x03_P2.54mm_Vertical, B.Cu at (128.2, 95.3)
- added J5: SM04B-GHS-TB, Connector_JST:JST_GH_SM04B-GHS-TB_1x04-1MP_P1.25mm_Horizontal, F.Cu at (119.8, 105.0)
- added R10: 100K, Resistor_SMD:R_0603_1608Metric, F.Cu at (120.2, 84.4)
- added R11: 100K, Resistor_SMD:R_0603_1608Metric, F.Cu at (185.2, 103.2)
- added R12: 10K, Resistor_SMD:R_0603_1608Metric, F.Cu at (159.6, 106.0)
- added R13: 100K, Resistor_SMD:R_0603_1608Metric, F.Cu at (176.0, 114.8)
- added R14: 10K, Resistor_SMD:R_0603_1608Metric, F.Cu at (144.2, 104.0)
- added R15: 4.99K, Resistor_SMD:R_0603_1608Metric, F.Cu at (147.4, 105.6)
- added R17: 1K, Resistor_SMD:R_0603_1608Metric, F.Cu at (159.4, 98.4)
- added R18: 1K, Resistor_SMD:R_0603_1608Metric, F.Cu at (147.4, 102.2)
- added R2: 2.2K, Resistor_SMD:R_0603_1608Metric, F.Cu at (162.6, 124.0)
- added R5: 100K, Resistor_SMD:R_0603_1608Metric, F.Cu at (162.6, 127.6)
- added R6: 1K, Resistor_SMD:R_0603_1608Metric, F.Cu at (171.2, 114.6)
- added R7: LDR07, OptoDevice:R_LDR_5.1x4.3mm_P3.4mm_Vertical, B.Cu at (118.3, 87.8)
- added R8: LDR07, OptoDevice:R_LDR_5.1x4.3mm_P3.4mm_Vertical, B.Cu at (188.3, 102.2)
- added R9: 10K, Resistor_SMD:R_0603_1608Metric, F.Cu at (183.8, 94.8)
- added TH1: 10K, Resistor_SMD:R_0603_1608Metric, F.Cu at (183.8, 98.8)
- added TH2: 10K, Resistor_SMD:R_0603_1608Metric, F.Cu at (163.4, 108.2)
- added U3: AD8676xR, Package_SO:SOIC-8_3.9x4.9mm_P1.27mm, F.Cu at (142.4, 98.8)
- added Y1: 8MHz, Crystal:Resonator_SMD_Murata_CSTxExxV-3Pin_3.0x1.1mm_HandSoldering, F.Cu at (167.2, 115.8)
- D1: value SFH203 -> 2200K; footprint LED_THT:LED_D5.0mm_IRGrey -> LED_SMD:LED_PLCC_2835_Handsoldering; moved to B.Cu
- D2: moved to B.Cu
- J1: value Motion -> ICSP; footprint Connector_PinSocket_2.54mm:PinSocket_1x03_P2.54mm_Vertical -> Connector_PinSocket_2.00mm:PinSocket_2x03_P2.00mm_Vertical
- J2: value FTDI -> SM04B-GHS-TB; footprint Connector_PinHeader_2.54mm:PinHeader_1x06_P2.54mm_Vertical -> Connector_JST:JST_GH_SM04B-GHS-TB_1x04-1MP_P1.25mm_Horizontal
- Q1: value QM6006D -> SiS454DN; footprint Package_TO_SOT_SMD:TO-252-2 -> Package_SO:Vishay_PowerPAK_1212-8_Single
- R1: value R_Shunt_US -> 2.2K; footprint Resistor_SMD:R_Shunt_Vishay_WSK2512_6332Metric_T1.19mm -> Resistor_SMD:R_0603_1608Metric
- TP1: value TestPoint -> 5016
- TP5: value 5016 -> TestPoint; footprint jannett_footprints:TestPoint_Keystone_5016_Compact -> jannett_footprints:TestPoint_Keystone_5016_Vias
- U1: value ESP32-WROOM-32E -> DS3231M; footprint RF_Module:ESP32-WROOM-32D -> Package_SO:SOIC-16W_7.5x10.3mm_P1.27mm
- U2: value AD8606ARZ -> ATmega328PB-A; footprint Package_SO:SOIC-8_3.9x4.9mm_P1.27mm -> Package_QFP:TQFP-32_7x7mm_P0.8mm
- moved PS1 98.8 mm to (132.2, 68.1)
- moved TP5 84.7 mm to (185.5, 88.1)
- moved TP2 79.4 mm to (163.4, 61.6)
- moved U1 66.7 mm to (158.0, 115.8), turned to -90 degrees
- moved Q1 66.2 mm to (155.0, 100.0), turned to 180 degrees
- moved TP4 65.1 mm to (170.1, 94.9)
- moved D2 63.1 mm to (160.0, 86.0), turned to 60 degrees
- moved TP3 61.6 mm to (124.8, 75.8)
- moved J2 57.9 mm to (187.9, 110.9), turned to 65 degrees
- moved TP6 56.9 mm to (133.6, 97.8)
- moved J1 55.6 mm to (182.4, 119.0), turned to -45 degrees
- moved D1 42.5 mm to (155.0, 85.0), turned to 90 degrees
- moved TP1 42.4 mm to (155.0, 95.0)
- moved U2 41.7 mm to (173.0, 107.8)
- moved R1 39.4 mm to (160.6, 124.0), turned to 90 degrees
Connections:
- D1 pad 1: unconnected-(D1-K-Pad1) -> VDD
- D1 pad 2: unconnected-(D1-A-Pad2) -> +3.3V
- D2 pad 1: Net-(D2-K) -> VDD
- J1 pad 1: +3.3V -> /MISO
- J1 pad 2: Net-(J1-Pin_2) -> +3.3V
- J1 pad 3: GND -> /SCK
- J2 pad 1: unconnected-(J2-Pin_1-Pad1) -> /ADC0
- J2 pad 2: unconnected-(J2-Pin_2-Pad2) -> GND
- J2 pad 3: unconnected-(J2-Pin_3-Pad3) -> /ADC1
- J2 pad 4: unconnected-(J2-Pin_4-Pad4) -> GND
- Q1 pad 1: Net-(Q1-G) -> GND
- Q1 pad 2: unconnected-(Q1-D-Pad2) -> GND
- Q1 pad 3: Net-(Q1-S) -> GND
- R1 pad 1: Net-(Q1-S) -> +3.3V
- R1 pad 2: unconnected-(R1-Pad2) -> /SDA
- TP1 pad 1: Net-(PS1-AC/L) -> VDD
- TP2 pad 1: Net-(PS1-AC/N) -> Net-(F1-Pad1)
- TP3 pad 1: +3.3V -> Net-(PS1-AC/N)
- TP4 pad 1: GND -> +3.3V
- TP5 pad 1: Net-(J1-Pin_2) -> GND
- TP6 pad 1: Net-(D2-K) -> /MOTION
- U1 pad 1: GND -> unconnected-(U1-32KHZ-Pad1)
- U1 pad 10: unconnected-(U1-IO25-Pad10) -> GND
- U1 pad 11: unconnected-(U1-IO26-Pad11) -> GND
- U1 pad 12: unconnected-(U1-IO27-Pad12) -> GND
- U1 pad 13: unconnected-(U1-IO14-Pad13) -> GND
- U1 pad 14: unconnected-(U1-IO12-Pad14) -> Net-(BT1-+)
- U1 pad 15: GND -> /SDA
- U1 pad 16: unconnected-(U1-IO13-Pad16) -> /SCL
- U1 pad 5: unconnected-(U1-SENSOR_VN-Pad5) -> GND
- U1 pad 6: unconnected-(U1-IO34-Pad6) -> GND
- U1 pad 7: unconnected-(U1-IO35-Pad7) -> GND
- U1 pad 8: unconnected-(U1-IO32-Pad8) -> GND
- U1 pad 9: unconnected-(U1-IO33-Pad9) -> GND
- U2 pad 1: Net-(Q1-G) -> /MOTION
- U2 pad 4: GND -> +3.3V
- U2 pad 5: unconnected-(U2B-+-Pad5) -> GND
- U2 pad 7: unconnected-(U2-Pad7) -> Net-(U2-XTAL1/PB6)
- U2 pad 8: unconnected-(U2C-V+-Pad8) -> Net-(U2-XTAL2/PB7)
Routing:
- net GND: track 0.00 -> 106.2 mm, vias 0 -> 1
- net +3.3V: track 0.00 -> 58.0 mm
- net Net-(U3A-+): track 0.00 -> 54.1 mm, vias 0 -> 2
- net Net-(C9-Pad1): track 0.00 -> 25.5 mm
- net /ADC0: track 0.00 -> 19.4 mm
- net /ADC1: track 0.00 -> 16.8 mm
- net Net-(U3A--): track 0.00 -> 16.3 mm, vias 0 -> 2
- net /MOTION: track 0.00 -> 15.0 mm
- net Net-(BT1-+): track 0.00 -> 14.1 mm
- net Net-(J3-Pin_3): track 0.00 -> 10.8 mm
- net Net-(U2-XTAL1/PB6): track 0.00 -> 7.93 mm
- net Net-(C7-Pad1): track 0.00 -> 7.65 mm
- net Net-(U2-XTAL2/PB7): track 0.00 -> 7.01 mm
- net /ADC3: track 0.00 -> 4.42 mm
- net Net-(U3B--): track 0.00 -> 4.38 mm
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- added copper zone on B.Cu, net +3.3V
- added copper zone on F.Cu, net +3.3V
- added copper zone on B.Cu, net GND
- added copper zone on F.Cu, net GND
- added copper zone on F.Cu, net VDD
Other:
- board outline added: 80 x 80 mm

Commit message: done
Parts:
- added REF**: Symbol_HighVoltage_Triangle_6x6mm_Copper, Symbol:Symbol_HighVoltage_Triangle_6x6mm_Copper, F.Cu at (126.4, 81.9)
- added REF**: Symbol_HighVoltage_Triangle_6x6mm_Copper, Symbol:Symbol_HighVoltage_Triangle_6x6mm_Copper, F.Cu at (169.8, 61.3)
- added REF**: Symbol_HighVoltage_Triangle_8x7mm_Copper, Symbol:Symbol_HighVoltage_Triangle_8x7mm_Copper, B.Cu at (132.7, 80.6)
- PS1: value IRM-20-3.3 -> LD15-23B03R2; footprint Converter_ACDC:Converter_ACDC_MeanWell_IRM-20-xx_THT -> jannett_footprints:LD15-23BxxR2_MNS
- moved PS1 9.48 mm to (135.6, 77.0)
Routing:
- net +3.3V: track 58.0 -> 223.7 mm, vias 0 -> 4
- net /ADC0: track 19.4 -> 137.5 mm, vias 0 -> 2
- net /RESET: track 1.60 -> 58.7 mm, vias 0 -> 2
- net /MOTION: track 15.0 -> 59.7 mm, vias 0 -> 2
- net Net-(BT1-+): track 14.1 -> 50.1 mm
- net /SCL: track 2.78 -> 29.1 mm, vias 0 -> 2
- net /SDA: track 2.96 -> 28.7 mm, vias 0 -> 2
- net /TX: track 2.73 -> 26.0 mm, vias 0 -> 2
- net /RX: track 2.93 -> 24.5 mm, vias 0 -> 2
- net GND: track 106.2 -> 125.5 mm, vias 1 -> 16
- net Net-(F1-Pad1): track 0.00 -> 18.5 mm
- net Net-(PS1-AC/L): track 0.00 -> 18.1 mm
- net Net-(PS1-AC/N): track 0.00 -> 16.7 mm
- net /SCK: track 0.00 -> 16.4 mm
- net /ADC3: track 4.42 -> 19.7 mm
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Other:
- board text added: "3.3V"
- board text added: "A0"
- board text added: "A1"
- board text added: "AC L"
- board text added: "AC N"
- board text added: "CAUTION HIGH VOLTAGE!!!"
- board text added: "Did you know? The Barred Owl’s call sounds like it's asking, “Who cooks for you?” — The perfect night watch companion for your porch!"
- board text added: "Dusk Lamp"
- board text added: "GND"
- board text added: "Jannett W"
- board text added: "MISO"
- board text added: "MOSI"
- board text added: "MOTION"
- board text added: "NC"
- board text added: "RST"
- board text added: "RX"
- board text added: "SCK"
- board text added: "TX"
- board text added: "VDD"
- board text added: "{dblquote}Smart light with wise company.{dblquote}"
